Commit message: Better implementation of inertia for the chasis and wheels. Doesn't entirely fix the problem however

File: urdf/actuators/wheels.xacro (robot description, xacro)
@@ -4,15 +4,14 @@
   <xacro:property name="wheel_radius" value="0.1"/>
   <xacro:property name="wheel_length" value="0.1"/>
-  <!-- <xacro:property name="wheel_rpy" value="1.55 0.0 0.0"/> -->
   <xacro:property name="wheel_rpy" value="1.57075 0 0"/>
-  <!-- <xacro:property name="wheel_rpy" value="0 0 0"/> -->
+  <xacro:property name="wheel_mass" value="2.0"/>
+  <xacro:property name="ixx" value="${1/12 * wheel_mass * (wheel_length * wheel_length)}"/>
+  <xacro:property name="izz" value="${1/12 * wheel_mass * (wheel_length * wheel_length)}"/>
   <xacro:macro name="wheel" params="side position flip alt">
     <xacro:property name="wheel_xyz" value="${alt * 0.3} ${flip * 0.2} -0.25"/>
     <link name="wheel_${side}_${position}">
       <inertial>
-        <!-- <origin xyz="0.0 0.0 0.0" rpy="0.0 0.0 0.0"/> -->
-        <!-- <mass value="1.0"/> -->
-        <mass value="3.0"/>
-        <inertia ixx="1.0" ixy="0.0" ixz="0.0" iyy="1.0" iyz="0.0" izz="1.0"/>
+        <mass value="${wheel_mass}"/>
+        <inertia ixx="${ixx}" ixy="0.0" ixz="0.0" iyy="0.0" iyz="0.0" izz="${izz}"/>
       </inertial>
       <visual name="">

File: urdf/cleaner.xacro (robot description, xacro)
@@ -8,10 +8,13 @@
   <xacro:property name="chasis_heigth" value="0.45"/>
   <xacro:property name="chasis_width" value="0.5"/>
+  <xacro:property name="chasis_mass" value="15.0"/>
+  <xacro:property name="ixx" value="${(1/12 * chasis_mass) * ((chasis_heigth * chasis_heigth) + (chasis_length * chasis_length))}"/>
+  <xacro:property name="iyy" value="${(1/12 * chasis_mass) * ((chasis_width * chasis_width) + (chasis_length * chasis_length))}"/>
+  <xacro:property name="izz" value="${(1/12 * chasis_mass) * ((chasis_width * chasis_width) + (chasis_heigth * chasis_heigth))}"/>
   <link name="chasis">
     <inertial>
-      <origin xyz="0.0 0.0 0.0" rpy="0.0 0.0 0.0"/>
-      <!-- <mass value="1.0"/> -->
-      <mass value="15.0"/>
-      <inertia ixx="0.4" ixy="0.0" ixz="0.0" iyy="0.4" iyz="0.0" izz="0.2"/>
+      <origin xyz="0.0 0.0 0.0" rpy="0.0 1.57 0.0"/>
+      <mass value="${chasis_mass}"/>
+      <inertia ixx="${ixx}" ixy="0.0" ixz="0.0" iyy="${iyy}" iyz="0.0" izz="${izz}"/>
     </inertial>
     <visual name="">
@@ -22,5 +25,4 @@
       <material name="">
         <color rgba="0.0 1.0 0.0 1.0"/>
-        <!-- <texture filename=""/> -->
       </material>
     </visual>
@@ -54,4 +56,5 @@
   <!-- MULTI-CAMERA -->
   <xacro:sweeper_cams/>
+  <xacro:overwatch_cam/>
   <!-- <xacro:sweeper_cam/> -->
   <!--  -->

File: urdf/sensors/camera.xacro (robot description, xacro)
@@ -107,3 +107,72 @@
         </joint>
     </xacro:macro>
+    <!-- overwatch camara -->
+    <xacro:macro name="overwatch_cam" params="">
+        <xacro:property name="overwatch_camera_link" value="0.3"/>
+        <!-- over-watch camera -->
+        <gazebo reference="overwatch_camara">
+            <sensor type="camera" name="camera1">
+                <update_rate>30.0</update_rate>
+                <camera name="test">
+                    <horizontal_fov>1.3962634</horizontal_fov>
+                    <image>
+                        <width>800</width>
+                        <height>800</height>
+                        <format>R8G8B8</format>
+                    </image>
+                    <clip>
+                        <near>0.02</near>
+                        <far>300</far>
+                    </clip>
+                    <noise>
+                        <type>gaussian</type>
+                        <!-- Noise is sampled independently per pixel on each frame.
+               That pixel's noise value is added to each of its color
+               channels, which at that point lie in the range [0,1]. -->
+                        <mean>0.0</mean>
+                        <stddev>0.007</stddev>
+                    </noise>
+                </camera>
+                <plugin name="camera_controller" filename="libgazebo_ros_camera.so">
+                    <alwaysOn>true</alwaysOn>
+                    <updateRate>0.0</updateRate>
+                    <cameraName>sweeper/camera1</cameraName>
+                    <imageTopicName>image_raw</imageTopicName>
+                    <cameraInfoTopicName>camera_info</cameraInfoTopicName>
+                    <frameName>overwatch_camara</frameName>
+                    <hackBaseline>0.07</hackBaseline>
+                    <distortionK1>0.0</distortionK1>
+                    <distortionK2>0.0</distortionK2>
+                    <distortionK3>0.0</distortionK3>
+                    <distortionT1>0.0</distortionT1>
+                    <distortionT2>0.0</distortionT2>
+                </plugin>
+            </sensor>
+        </gazebo>
+        <link name="overwatch_camara">
+            <inertial>
+                <origin xyz="0.0 0.0 0.0" rpy="0.0 0.0 0.0"/>
+                <mass value="0.0"/>
+                <inertia ixx="0.0" ixy="0.0" ixz="0.0" iyy="0.0" iyz="0.0" izz="0.0"/>
+            </inertial>
+            <visual name="">
+                <origin xyz="0.0 0.0 0.0" rpy="0.0 0.0 0.0"/>
+                <geometry>
+                    <!-- <mesh filename="package://sweep_bot/meshes/model.sdf"/> -->
+                    <box size="0.0 0.0 0.0"/>
+                </geometry>
+            </visual>
+            <collision>
+                <origin xyz="0.0 0.0 0.0" rpy="0.0 0.0 0.0"/>
+                <geometry>
+                    <box size="0.0 0.0 0.0"/>
+                </geometry>
+            </collision>
+        </link>
+        <joint name="overwatch_joint" type="fixed">
+            <origin xyz="-3.0 ${chasis_width / 1.85} 1.5" rpy="0.0 0.0 0.0"/>
+            <parent link="chasis"/>
+            <child link="overwatch_camara"/>
+        </joint>
+    </xacro:macro>
 </robot>
