Commit message: Updates to the mapping launch file - for attempting to map the streets Creates the scan_merge launch file - for separate initialization of the laserscan_multi_merger node otherwise merge process doesn't work Updates to cleaner and laser xacro files

File: urdf/cleaner.xacro (robot description, xacro)
@@ -4,4 +4,5 @@
   <xacro:include filename="$(find sweep_bot)/urdf/actuators/wheels.xacro"/>
   <xacro:include filename="$(find sweep_bot)/urdf/sensors/MultiCamera.xacro"/>
+  <xacro:include filename="$(find sweep_bot)/urdf/sensors/laser.xacro"/>
   <!-- body -->
   <xacro:property name="chasis_length" value="1.0"/>
@@ -50,12 +51,14 @@
   </VLP-16> -->
   <!-- os1_sensor_mount_joint -->
-  <xacro:include filename="$(find ouster_description)/urdf/OS1-64.urdf.xacro"/>
+  <!-- <xacro:include filename="$(find ouster_description)/urdf/OS1-64.urdf.xacro"/>
   <OS1-64 parent="chasis" name="os1_sensor" hz="10" samples="220">
     <origin xyz="0 0 0.3" rpy="0 0 0" />
-  </OS1-64>
+  </OS1-64> -->
   <!-- MULTI-CAMERA -->
   <xacro:sweeper_cams/>
   <xacro:overwatch_cam/>
-  <!-- <xacro:sweeper_cam/> -->
+  <!-- <xacro:laser_top/> -->
+  <xacro:laser_left/>
+  <xacro:laser_right/>
   <!--  -->
   <!-- <gazebo>
@@ -96,4 +99,10 @@
       <topicName>cmd_vel</topicName>
       <broadcastTF>true</broadcastTF>
+      <commandTopic> cmd_vel </commandTopic>
+      <odometryTopic> odom </odometryTopic>
+      <odometryFrame> odom </odometryFrame>
+      <covariance_x> 0.000100 </covariance_x>
+      <covariance_y> 0.000100 </covariance_y>
+      <covariance_yaw> 0.010000 </covariance_yaw>
     </plugin>
   </gazebo>

File: urdf/sensors/laser.xacro (robot description, xacro)
@@ -1,7 +1,38 @@
 <?xml version="1.0"?>
 <robot xmlns:xacro="http://www.ros.org/wiki/xacro" name="robot_name">
-    <xacro:macro name="laser">
-        <!-- Hokuyo Laser -->
-        <link name="hokuyo_link">
+    <!-- <xacro:macro name="laser_top">
+        <gazebo reference="hokuyo_link_top">
+            <sensor type="ray" name="head_hokuyo_sensor">
+            <pose>0 0 0 0 0 0</pose>
+            <visualize>false</visualize>
+            <update_rate>20</update_rate>
+            <ray>
+                <scan>
+                    <horizontal>
+                        <samples>720</samples>
+                        <resolution>1</resolution>
+                        <min_angle>-1.570796</min_angle>
+                        <max_angle>1.570796</max_angle>
+                    </horizontal>
+                </scan>
+                <range>
+                    <min>0.10</min>
+                    <max>10.0</max>
+                    <resolution>0.05</resolution>
+                </range>
+                <noise>
+                    <type>gaussian</type>
+                    <mean>0.0</mean>
+                    <stddev>0.01</stddev>
+                </noise>
+            </ray>
+            <plugin name="gazebo_ros_head_hokuyo_controller" filename="libgazebo_ros_laser.so">
+                <topicName>/scan</topicName>
+                <frameName>hokuyo_link_top</frameName>
+            </plugin>
+            </sensor>
+        </gazebo> -->
+        <!-- Hokuyo Laser - TOP -->
+        <link name="hokuyo_link_top">
             <collision>
                 <origin xyz="0 0 0" rpy="0 0 0"/>
@@ -22,9 +53,154 @@
             </inertial>
         </link>
-        <joint name="laser_joint" type="fixed">
-            <origin xyz="0.0 0.0 0.29" rpy="0.0 0.0 0.0"/>
+        <joint name="laser_joint_top" type="fixed">
+            <origin xyz="0.0 0 0.29" rpy="0 0 0"/>
             <parent link="chasis"/>
-            <child link="hokuyo_link"/>
+            <child link="hokuyo_link_top"/>
+        </joint>
+    <!-- </xacro:macro> -->
+    <!-- Hokuyo Laser - LEFT -->
+    <xacro:macro name="laser_left">
+        <gazebo reference="hokuyo_link_left">
+            <sensor type="ray" name="head_hokuyo_sensor">
+            <pose>0 0 0 0 0 0</pose>
+            <visualize>true</visualize>
+            <update_rate>20</update_rate>
+            <ray>
+                <scan>
+                    <horizontal>
+                        <samples>720</samples>
+                        <resolution>1</resolution>
+                        <min_angle>-1.570796</min_angle>
+                        <max_angle>1.570796</max_angle>
+                    </horizontal>
+                </scan>
+                <range>
+                    <min>0.10</min>
+                    <max>10.0</max>
+                    <resolution>0.05</resolution>
+                </range>
+                <noise>
+                    <type>gaussian</type>
+                    <mean>0.0</mean>
+                    <stddev>0.01</stddev>
+                </noise>
+            </ray>
+            <plugin name="gazebo_ros_head_hokuyo_controller" filename="libgazebo_ros_laser.so">
+                <topicName>/scan_left</topicName>
+                <frameName>hokuyo_link_left</frameName>
+            </plugin>
+            </sensor>
+        </gazebo>
+        <!--  -->
+        <link name="hokuyo_link_left">
+            <collision>
+                <origin xyz="0 0 0" rpy="0 0 0"/>
+                <geometry>
+                    <box size="0.1 0.1 0.1"/>
+                </geometry>
+            </collision>
+            <visual>
+                <origin xyz="0 0 0" rpy="0 0 0"/>
+                <geometry>
+                    <mesh filename="package://rrbot_description/meshes/hokuyo.dae"/>
+                </geometry>
+            </visual>
+            <inertial>
+                <mass value="1e-5" />
+                <origin xyz="0 0 0" rpy="0 0 0"/>
+                <inertia ixx="1e-6" ixy="0" ixz="0" iyy="1e-6" iyz="0" izz="1e-6" />
+            </inertial>
+        </link>
+        <joint name="laser_joint_left" type="fixed">
+            <!-- <origin xyz="0.0 0.25 0.29" rpy="-0.5 0 0"/> -->
+            <origin xyz="0.0 0.27 -0.20" rpy="0 0 0"/>
+            <parent link="chasis"/>
+            <child link="hokuyo_link_left"/>
         </joint>
     </xacro:macro>
+    <!-- Hokuyo Laser - RIGHT -->
+    <xacro:macro name="laser_right">
+        <gazebo reference="hokuyo_link_right">
+            <sensor type="ray" name="head_hokuyo_sensor">
+            <pose>0 0 0 0 0 0</pose>
+            <visualize>true</visualize>
+            <update_rate>20</update_rate>
+            <ray>
+                <scan>
+                    <horizontal>
+                        <samples>720</samples>
+                        <resolution>1</resolution>
+                        <min_angle>-1.570796</min_angle>
+                        <max_angle>1.570796</max_angle>
+                    </horizontal>
+                </scan>
+                <range>
+                    <min>0.10</min>
+                    <max>10.0</max>
+                    <resolution>0.05</resolution>
+                </range>
+                <noise>
+                    <type>gaussian</type>
+                    <mean>0.0</mean>
+                    <stddev>0.01</stddev>
+                </noise>
+            </ray>
+            <plugin name="gazebo_ros_head_hokuyo_controller" filename="libgazebo_ros_laser.so">
+                <topicName>/scan_right</topicName>
+                <frameName>hokuyo_link_right</frameName>
+            </plugin>
+            </sensor>
+        </gazebo>
+        <!--  -->
+        <link name="hokuyo_link_right">
+            <collision>
+                <origin xyz="0 0 0" rpy="0 0 0"/>
+                <geometry>
+                    <box size="0.1 0.1 0.1"/>
+                </geometry>
+            </collision>
+            <visual>
+                <origin xyz="0 0 0" rpy="0 0 0"/>
+                <geometry>
+                    <mesh filename="package://rrbot_description/meshes/hokuyo.dae"/>
+                </geometry>
+            </visual>
+            <inertial>
+                <mass value="1e-5" />
+                <origin xyz="0 0 0" rpy="0 0 0"/>
+                <inertia ixx="1e-6" ixy="0" ixz="0" iyy="1e-6" iyz="0" izz="1e-6" />
+            </inertial>
+        </link>
+        <joint name="laser_joint_right" type="fixed">
+            <!-- <origin xyz="0.0 -0.25 0.29" rpy="0.5 0 0"/> -->
+            <!-- <origin xyz="0.0 -0.27 -0.20" rpy="0 0 0"/> -->
+            <!-- <origin xyz="0.0 0 0" rpy="0 0 0"/> -->
+            <origin xyz="0.0 -0.27 -0.20" rpy="0 0 0"/>
+            <parent link="chasis"/>
+            <child link="hokuyo_link_right"/>
+        </joint>
+    </xacro:macro>
+    <!-- test -->
+    <!-- <xacro:macro name="laser_right">
+    <link name="hokuyo_link_right">
+        <visual>
+            <origin xyz="0 0 0" rpy="0 0 0"/>
+            <geometry>
+                <mesh filename="package://rrbot_description/meshes/hokuyo.dae"/>
+            </geometry>
+        </visual>
+        <inertial>
+        <mass value="0.000001" />
+        <origin xyz="0 0 0" />
+        <inertia ixx="0.0001" ixy="0.0" ixz="0.0"
+            iyy="0.0001" iyz="0.0"
+            izz="0.0001" />
+        </inertial>
+    </link>
+    <joint name="laser" type="fixed">
+        <origin xyz="-0.005 0.00 0.360" rpy="3.14159 0 0" />
+        <parent link="chasis" />
+        <child link="hokuyo_link_right" />
+    </joint>
+    </xacro:macro> -->
 </robot>

Commit message: Gmapping related content - unsuccessful at creating a clean map of the city

File: urdf/cleaner.xacro (robot description, xacro)
@@ -46,8 +46,8 @@
   <!-- <xacro:VLP16 /> -->
   <!-- name="velodyne" topic="/velodyne_points" hz="10" lasers="16" samples="1875" collision_range="0.3" min_range="0.9" max_range="130.0" noise="0.008" min_angle="-${M_PI}" max_angle="${M_PI}" gpu="false"/> -->
-  <!-- <xacro:include filename="$(find velodyne_description)/urdf/VLP-16.urdf.xacro"/>
+  <xacro:include filename="$(find velodyne_description)/urdf/VLP-16.urdf.xacro"/>
   <VLP-16 parent="chasis" name="velodyne" topic="/velodyne_points" hz="10" samples="1000" gpu="10">
     <origin xyz="0 0 0.25" rpy="0 0 0" />
-  </VLP-16> -->
+  </VLP-16>
   <!-- os1_sensor_mount_joint -->
   <!-- <xacro:include filename="$(find ouster_description)/urdf/OS1-64.urdf.xacro"/>
@@ -58,7 +58,10 @@
   <xacro:sweeper_cams/>
   <xacro:overwatch_cam/>
+  <!-- LASERS -->
   <!-- <xacro:laser_top/> -->
-  <xacro:laser_left/>
-  <xacro:laser_right/>
+  <xacro:laser_front/>
+  <!-- <xacro:laser_left/> -->
+  <!-- <xacro:laser_right/> -->
+  <!-- <xacro:laser_rear/> -->
   <!--  -->
   <!-- <gazebo>

File: urdf/sensors/laser.xacro (robot description, xacro)
@@ -1,9 +1,10 @@
 <?xml version="1.0"?>
 <robot xmlns:xacro="http://www.ros.org/wiki/xacro" name="robot_name">
-    <!-- <xacro:macro name="laser_top">
-        <gazebo reference="hokuyo_link_top">
+    <!-- Hokuyo Laser - TOP -->
+    <xacro:macro name="laser_top">
+        <!-- <gazebo reference="hokuyo_link_top">
             <sensor type="ray" name="head_hokuyo_sensor">
             <pose>0 0 0 0 0 0</pose>
-            <visualize>false</visualize>
+            <visualize>true</visualize>
             <update_rate>20</update_rate>
             <ray>
@@ -12,6 +13,6 @@
                         <samples>720</samples>
                         <resolution>1</resolution>
-                        <min_angle>-1.570796</min_angle>
-                        <max_angle>1.570796</max_angle>
+                        <min_angle>-0.5</min_angle>
+                        <max_angle>0.5</max_angle>
                     </horizontal>
                 </scan>
@@ -33,5 +34,4 @@
             </sensor>
         </gazebo> -->
-        <!-- Hokuyo Laser - TOP -->
         <link name="hokuyo_link_top">
             <collision>
@@ -58,9 +58,74 @@
             <child link="hokuyo_link_top"/>
         </joint>
-    <!-- </xacro:macro> -->
+    </xacro:macro>
+    <!-- Hokuyo Laser - FRONT -->
+    <xacro:macro name="laser_front">
+        <gazebo reference="hokuyo_link_front">
+            <sensor type="ray" name="head_hokuyo_sensor_front">
+            <pose>0 0 0 0 0 0</pose>
+            <visualize>true</visualize>
+            <!-- <update_rate>20</update_rate> -->
+            <update_rate>50</update_rate>
+            <ray>
+                <scan>
+                    <horizontal>
+                        <samples>720</samples>
+                        <resolution>1</resolution>
+                        <!-- <min_angle>-1.570796</min_angle> -->
+                        <!-- <max_angle>1.570796</max_angle> -->
+                        <min_angle>-1.5</min_angle>
+                        <max_angle>1.5</max_angle>
+                    </horizontal>
+                </scan>
+                <range>
+                    <min>0.10</min>
+                    <max>25</max>
+                    <resolution>0.05</resolution>
+                </range>
+                <noise>
+                    <type>gaussian</type>
+                    <mean>0.0</mean>
+                    <stddev>0.01</stddev>
+                </noise>
+            </ray>
+            <plugin name="gazebo_ros_head_hokuyo_controller" filename="libgazebo_ros_laser.so">
+                <topicName>/scan</topicName>
+                <frameName>hokuyo_link_front</frameName>
+            </plugin>
+            </sensor>
+        </gazebo>
+        <!--  -->
+        <link name="hokuyo_link_front">
+            <collision>
+                <origin xyz="0 0 0" rpy="0 0 0"/>
+                <geometry>
+                    <box size="0.1 0.1 0.1"/>
+                </geometry>
+            </collision>
+            <visual>
+                <origin xyz="0 0 0" rpy="0 0 0"/>
+                <geometry>
+                    <mesh filename="package://rrbot_description/meshes/hokuyo.dae"/>
+                </geometry>
+            </visual>
+            <inertial>
+                <mass value="1e-5" />
+                <origin xyz="0 0 0" rpy="0 0 0"/>
+                <inertia ixx="1e-6" ixy="0" ixz="0" iyy="1e-6" iyz="0" izz="1e-6" />
+            </inertial>
+        </link>
+        <joint name="laser_joint_front" type="fixed">
+            <!-- <origin xyz="0.53 0 -0.20" rpy="0 0.01 0"/> -->
+            <!-- <origin xyz="0.53 0 -0.25" rpy="0 0.0 0"/> -->
+            <!-- <origin xyz="0.53 0 -0.22" rpy="0 0.0 0"/> -->
+            <origin xyz="0.53 0 0" rpy="0 0.0 0"/>
+            <parent link="chasis"/>
+            <child link="hokuyo_link_front"/>
+        </joint>
+    </xacro:macro>
     <!-- Hokuyo Laser - LEFT -->
     <xacro:macro name="laser_left">
         <gazebo reference="hokuyo_link_left">
-            <sensor type="ray" name="head_hokuyo_sensor">
+            <sensor type="ray" name="head_hokuyo_sensor_left">
             <pose>0 0 0 0 0 0</pose>
             <visualize>true</visualize>
@@ -71,6 +136,8 @@
                         <samples>720</samples>
                         <resolution>1</resolution>
-                        <min_angle>-1.570796</min_angle>
-                        <max_angle>1.570796</max_angle>
+                        <!-- <min_angle>-1.570796</min_angle> -->
+                        <!-- <max_angle>1.570796</max_angle> -->
+                        <min_angle>-1.5</min_angle>
+                        <max_angle>1.5</max_angle>
                     </horizontal>
                 </scan>
@@ -114,5 +181,5 @@
         <joint name="laser_joint_left" type="fixed">
             <!-- <origin xyz="0.0 0.25 0.29" rpy="-0.5 0 0"/> -->
-            <origin xyz="0.0 0.27 -0.20" rpy="0 0 0"/>
+            <origin xyz="0.0 0.25 -0.20" rpy="0 0.01 ${3.14/2}"/>
             <parent link="chasis"/>
             <child link="hokuyo_link_left"/>
@@ -122,5 +189,5 @@
     <xacro:macro name="laser_right">
         <gazebo reference="hokuyo_link_right">
-            <sensor type="ray" name="head_hokuyo_sensor">
+            <sensor type="ray" name="head_hokuyo_sensor_right">
             <pose>0 0 0 0 0 0</pose>
             <visualize>true</visualize>
@@ -131,6 +198,8 @@
                         <samples>720</samples>
                         <resolution>1</resolution>
-                        <min_angle>-1.570796</min_angle>
-                        <max_angle>1.570796</max_angle>
+                        <!-- <min_angle>-1.570796</min_angle> -->
+                        <!-- <max_angle>1.570796</max_angle> -->
+                        <min_angle>-1.5</min_angle>
+                        <max_angle>1.5</max_angle>
                     </horizontal>
                 </scan>
@@ -173,34 +242,69 @@
         </link>
         <joint name="laser_joint_right" type="fixed">
-            <!-- <origin xyz="0.0 -0.25 0.29" rpy="0.5 0 0"/> -->
-            <!-- <origin xyz="0.0 -0.27 -0.20" rpy="0 0 0"/> -->
-            <!-- <origin xyz="0.0 0 0" rpy="0 0 0"/> -->
-            <origin xyz="0.0 -0.27 -0.20" rpy="0 0 0"/>
+            <origin xyz="0.0 -0.25 -0.20" rpy="0 0.01 -${3.14/2}"/>
             <parent link="chasis"/>
             <child link="hokuyo_link_right"/>
         </joint>
     </xacro:macro>
-    <!-- test -->
-    <!-- <xacro:macro name="laser_right">
-    <link name="hokuyo_link_right">
-        <visual>
-            <origin xyz="0 0 0" rpy="0 0 0"/>
-            <geometry>
-                <mesh filename="package://rrbot_description/meshes/hokuyo.dae"/>
-            </geometry>
-        </visual>
-        <inertial>
-        <mass value="0.000001" />
-        <origin xyz="0 0 0" />
-        <inertia ixx="0.0001" ixy="0.0" ixz="0.0"
-            iyy="0.0001" iyz="0.0"
-            izz="0.0001" />
-        </inertial>
-    </link>
-    <joint name="laser" type="fixed">
-        <origin xyz="-0.005 0.00 0.360" rpy="3.14159 0 0" />
-        <parent link="chasis" />
-        <child link="hokuyo_link_right" />
-    </joint>
-    </xacro:macro> -->
+    <!-- Hokuyo Laser - REAR -->
+    <xacro:macro name="laser_rear">
+        <gazebo reference="hokuyo_link_rear">
+            <sensor type="ray" name="head_hokuyo_sensor_rear">
+            <pose>0 0 0 0 0 0</pose>
+            <visualize>true</visualize>
+            <update_rate>20</update_rate>
+            <ray>
+                <scan>
+                    <horizontal>
+                        <samples>720</samples>
+                        <resolution>1</resolution>
+                        <!-- <min_angle>-1.570796</min_angle> -->
+                        <!-- <max_angle>1.570796</max_angle> -->
+                        <min_angle>-1.5</min_angle>
+                        <max_angle>1.5</max_angle>
+                    </horizontal>
+                </scan>
+                <range>
+                    <min>0.10</min>
+                    <max>10.0</max>
+                    <resolution>0.05</resolution>
+                </range>
+                <noise>
+                    <type>gaussian</type>
+                    <mean>0.0</mean>
+                    <stddev>0.01</stddev>
+                </noise>
+            </ray>
+            <plugin name="gazebo_ros_head_hokuyo_controller" filename="libgazebo_ros_laser.so">
+                <topicName>/scan_rear</topicName>
+                <frameName>hokuyo_link_rear</frameName>
+            </plugin>
+            </sensor>
+        </gazebo>
+        <!--  -->
+        <link name="hokuyo_link_rear">
+            <collision>
+                <origin xyz="0 0 0" rpy="0 0 0"/>
+                <geometry>
+                    <box size="0.1 0.1 0.1"/>
+                </geometry>
+            </collision>
+            <visual>
+                <origin xyz="0 0 0" rpy="0 0 0"/>
+                <geometry>
+                    <mesh filename="package://rrbot_description/meshes/hokuyo.dae"/>
+                </geometry>
+            </visual>
+            <inertial>
+                <mass value="1e-5" />
+                <origin xyz="0 0 0" rpy="0 0 0"/>
+                <inertia ixx="1e-6" ixy="0" ixz="0" iyy="1e-6" iyz="0" izz="1e-6" />
+            </inertial>
+        </link>
+        <joint name="laser_joint_rear" type="fixed">
+            <origin xyz="-0.53 0 -0.20" rpy="0 0.01 ${3.14}"/>
+            <parent link="chasis"/>
+            <child link="hokuyo_link_rear"/>
+        </joint>
+    </xacro:macro>
 </robot>
