Commit message: hector work in progress

File: urdf/cleaner.xacro (robot description, xacro)
@@ -5,12 +5,19 @@
   <xacro:include filename="$(find sweep_bot)/urdf/sensors/MultiCamera.xacro"/>
   <xacro:include filename="$(find sweep_bot)/urdf/sensors/laser.xacro"/>
+  <xacro:include filename="$(find hector_sensors_description)/urdf/hokuyo_utm30lx.urdf.xacro"/>
   <!-- body -->
   <xacro:property name="chasis_length" value="1.0"/>
-  <xacro:property name="chasis_heigth" value="0.45"/>
-  <xacro:property name="chasis_width" value="0.5"/>
+  <xacro:property name="chasis_width" value="0.45"/>
+  <xacro:property name="chasis_heigth" value="0.5"/>
   <xacro:property name="chasis_mass" value="15.0"/>
-  <xacro:property name="ixx" value="${(1/12 * chasis_mass) * ((chasis_heigth * chasis_heigth) + (chasis_length * chasis_length))}"/>
-  <xacro:property name="iyy" value="${(1/12 * chasis_mass) * ((chasis_width * chasis_width) + (chasis_length * chasis_length))}"/>
-  <xacro:property name="izz" value="${(1/12 * chasis_mass) * ((chasis_width * chasis_width) + (chasis_heigth * chasis_heigth))}"/>
+  <xacro:property name="ixx" value="${(1/12 * chasis_mass) * ((chasis_width * chasis_width) + (chasis_length * chasis_length))}"/>
+  <xacro:property name="iyy" value="${(1/12 * chasis_mass) * ((chasis_heigth * chasis_heigth) + (chasis_length * chasis_length))}"/>
+  <xacro:property name="izz" value="${(1/12 * chasis_mass) * ((chasis_heigth * chasis_heigth) + (chasis_width * chasis_width))}"/>
+  <link name="chasis_footprint"/>
+  <joint name="chasis_footprint_joint" type="fixed">
+    <parent link="chasis_footprint"/>
+    <child link="chasis"/>
+    <origin xyz="0.0 0.0 0.0" rpy="0.0 0.0 0.0"/>
+  </joint>
   <link name="chasis">
     <inertial>
@@ -22,5 +29,5 @@
       <origin xyz="0.0 0.0 0.0" rpy="0.0 0.0 0.0"/>
       <geometry>
-        <box size="${chasis_length} ${chasis_heigth} ${chasis_width}"/>
+        <box size="${chasis_length} ${chasis_width} ${chasis_heigth}"/>
       </geometry>
       <material name="">
@@ -31,5 +38,5 @@
       <origin xyz="0.0 0.0 0.0" rpy="0.0 0.0 0.0"/>
       <geometry>
-        <box size="${chasis_length} ${chasis_heigth} ${chasis_width}"/>
+        <box size="${chasis_length} ${chasis_width} ${chasis_heigth}"/>
       </geometry>
     </collision>
@@ -43,48 +50,17 @@
   <xacro:wheel side="left" position="aft" flip='1' alt='-1'/>
   <xacro:wheel side="right" position="aft" flip='-1' alt='-1'/>
-  <!-- LIDAR -->
-  <!-- <xacro:VLP16 /> -->
-  <!-- name="velodyne" topic="/velodyne_points" hz="10" lasers="16" samples="1875" collision_range="0.3" min_range="0.9" max_range="130.0" noise="0.008" min_angle="-${M_PI}" max_angle="${M_PI}" gpu="false"/> -->
-  <xacro:include filename="$(find velodyne_description)/urdf/VLP-16.urdf.xacro"/>
-  <VLP-16 parent="chasis" name="velodyne" topic="/velodyne_points" hz="10" samples="1000" gpu="10">
-    <origin xyz="0 0 0.25" rpy="0 0 0" />
-  </VLP-16>
-  <!-- os1_sensor_mount_joint -->
-  <!-- <xacro:include filename="$(find ouster_description)/urdf/OS1-64.urdf.xacro"/>
-  <OS1-64 parent="chasis" name="os1_sensor" hz="10" samples="220">
+  <!-- HOKUYO as RPLIDAR -->
+  <xacro:hokuyo_utm30lx name="hokuyo_laser" parent="chasis" ros_topic="hokuyo_scan" update_rate="40" ray_count="1040" min_angle="130" max_angle="-130">
     <origin xyz="0 0 0.3" rpy="0 0 0" />
-  </OS1-64> -->
+  </xacro:hokuyo_utm30lx>
   <!-- MULTI-CAMERA -->
   <xacro:sweeper_cams/>
-  <xacro:overwatch_cam/>
+  <!-- <xacro:overwatch_cam/> -->
   <!-- LASERS -->
-  <!-- <xacro:laser_top/> -->
-  <xacro:laser_front/>
-  <!-- <xacro:laser_left/> -->
-  <!-- <xacro:laser_right/> -->
+  <xacro:laser_top/>
+  <!-- <xacro:laser_front/> -->
+  <xacro:laser_left/>
+  <xacro:laser_right/>
   <!-- <xacro:laser_rear/> -->
-  <!--  -->
-  <!-- <gazebo>
-    <plugin filename="libgazebo_ros_diff_drive.so" name="differential_drive_controller_front">
-      <rosDebugLevel>Debug</rosDebugLevel>
-      <publishWheelTF>True</publishWheelTF>
-      <publishTf>1</publishTf>
-      <publishWheelJointState>true</publishWheelJointState>
-      <alwaysOn>true</alwaysOn>
-      <updateRate>100.0</updateRate>
-      <leftJoint>body_wheel_left_aft_joint</leftJoint>
-      <rightJoint>body_wheel_right_aft_joint</rightJoint>
-      <wheelSeparation>0.3</wheelSeparation>
-      <wheelDiameter>0.08</wheelDiameter>
-      <broadcastTF>1</broadcastTF>
-      <wheelTorque>30</wheelTorque>
-      <wheelAcceleration>1.8</wheelAcceleration>
-      <commandTopic>cmd_vel</commandTopic>
-      <odometryFrame>odom</odometryFrame>
-      <odometryTopic>odom</odometryTopic>
-      <robotBaseFrame>chasis</robotBaseFrame>
-    </plugin>
-  </gazebo> -->
-  <!--  -->
   <!-- SKIP STEERING -->
   <gazebo>
@@ -98,5 +74,5 @@
       <wheelSeparation>0.5</wheelSeparation>
       <wheelDiameter>0.2</wheelDiameter>
-      <robotBaseFrame>chasis</robotBaseFrame>
+      <robotBaseFrame>chasis_footprint</robotBaseFrame>
       <torque>20</torque>
       <topicName>cmd_vel</topicName>
@@ -112,8 +88,2 @@
   <!--  -->
 </robot>
-<!--
-  body_wheel_left_aft_joint
-  body_wheel_left_fore_joint
-  body_wheel_right_aft_joint
-  body_wheel_right_fore_joint
--->

File: urdf/sensors/MultiCamera.xacro (robot description, xacro)
@@ -46,5 +46,5 @@
                     <imageTopicName>image_raw</imageTopicName>
                     <cameraInfoTopicName>camera_info</cameraInfoTopicName>
-                    <frameName>right_camera</frameName>
+                    <frameName>left_camera_optical_frame</frameName>
                     <!--<rightFrameName>right_camera_optical_frame</rightFrameName>-->
                     <hackBaseline>0.07</hackBaseline>
@@ -57,5 +57,5 @@
             </sensor>
         </gazebo>
-        <!--  -->
+        <!-- CAMERA LEFT -->
         <link name="left_camera">
             <inertial>
@@ -82,5 +82,5 @@
         </link>
         <joint name="left_camera_joint" type="fixed">
-            <origin xyz="0.45 -${chasis_width / 1.82} 0.0" rpy="0.0 0.0 0.0"/>
+            <origin xyz="0.45 -${chasis_heigth / 1.82} 0.0" rpy="0.0 0.0 0.0"/>
             <parent link="chasis"/>
             <child link="left_camera"/>
@@ -88,4 +88,5 @@
             <!-- <limit lower="0.0" upper="0.0" effort="0.0" velocity="0.0"/> -->
         </joint>
+        <!-- CAMERA RIGHT -->
         <link name="right_camera">
             <inertial>
@@ -112,5 +113,5 @@
         </link>
         <joint name="right_camera_joint" type="fixed">
-            <origin xyz="0.45 ${chasis_width / 1.82} 0.0" rpy="0.0 0.0 0.0"/>
+            <origin xyz="0.45 ${chasis_heigth / 1.82} 0.0" rpy="0.0 0.0 0.0"/>
             <parent link="chasis"/>
             <child link="right_camera"/>

Commit message: Successfully generated usable map using Hector Now working on wall following

File: urdf/cleaner.xacro (robot description, xacro)
@@ -60,5 +60,5 @@
   <!-- <xacro:laser_top/> -->
   <!-- <xacro:laser_front/> -->
-  <!-- <xacro:laser_left/> -->
+  <xacro:laser_left/>
   <!-- <xacro:laser_right/> -->
   <!-- <xacro:laser_rear/> -->

File: urdf/sensors/laser.xacro (robot description, xacro)
@@ -66,9 +66,9 @@
             <visualize>true</visualize>
             <!-- <update_rate>20</update_rate> -->
-            <update_rate>50</update_rate>
-            <ray>
-                <scan>
-                    <horizontal>
-                        <samples>720</samples>
+            <update_rate>20</update_rate>
+            <ray>
+                <scan>
+                    <horizontal>
+                        <samples>50</samples>
                         <resolution>1</resolution>
                         <!-- <min_angle>-1.570796</min_angle> -->
@@ -80,15 +80,15 @@
                 <range>
                     <min>0.10</min>
-                    <max>25</max>
-                    <resolution>0.05</resolution>
-                </range>
-                <noise>
-                    <type>gaussian</type>
-                    <mean>0.0</mean>
-                    <stddev>0.01</stddev>
-                </noise>
-            </ray>
-            <plugin name="gazebo_ros_head_hokuyo_controller" filename="libgazebo_ros_laser.so">
-                <topicName>/scan</topicName>
+                    <max>10</max>
+                    <resolution>0.05</resolution>
+                </range>
+                <noise>
+                    <type>gaussian</type>
+                    <mean>0.0</mean>
+                    <stddev>0.01</stddev>
+                </noise>
+            </ray>
+            <plugin name="gazebo_ros_head_hokuyo_controller" filename="libgazebo_ros_laser.so">
+                <topicName>/scan_front</topicName>
                 <frameName>hokuyo_link_front</frameName>
             </plugin>
@@ -116,8 +116,8 @@
         </link>
         <joint name="laser_joint_front" type="fixed">
-            <!-- <origin xyz="0.53 0 -0.20" rpy="0 0.01 0"/> -->
+            <origin xyz="0.53 0 -0.20" rpy="0 0.0 0"/>
             <!-- <origin xyz="0.53 0 -0.25" rpy="0 0.0 0"/> -->
             <!-- <origin xyz="0.53 0 -0.22" rpy="0 0.0 0"/> -->
-            <origin xyz="0.53 0 0" rpy="0 0.0 0"/>
+            <!-- <origin xyz="0.53 0 0" rpy="0 0.0 0"/> -->
             <parent link="chasis"/>
             <child link="hokuyo_link_front"/>
@@ -134,5 +134,69 @@
                 <scan>
                     <horizontal>
-                        <samples>720</samples>
+                        <samples>50</samples>
+                        <resolution>1</resolution>
+                        <!-- <min_angle>-1.570796</min_angle> -->
+                        <!-- <max_angle>1.570796</max_angle> -->
+                        <!-- <min_angle>-1.5</min_angle> -->
+                        <!-- <max_angle>1.5</max_angle> -->
+                        <min_angle>-0.2</min_angle>
+                        <max_angle>0.2</max_angle>
+                    </horizontal>
+                </scan>
+                <range>
+                    <min>0.10</min>
+                    <max>10.0</max>
+                    <resolution>0.05</resolution>
+                </range>
+                <noise>
+                    <type>gaussian</type>
+                    <mean>0.0</mean>
+                    <stddev>0.01</stddev>
+                </noise>
+            </ray>
+            <plugin name="gazebo_ros_head_hokuyo_controller" filename="libgazebo_ros_laser.so">
+                <topicName>/scan_left</topicName>
+                <frameName>hokuyo_link_left</frameName>
+            </plugin>
+            </sensor>
+        </gazebo>
+        <!--  -->
+        <link name="hokuyo_link_left">
+            <collision>
+                <origin xyz="0 0 0" rpy="0 0 0"/>
+                <geometry>
+                    <box size="0.1 0.1 0.1"/>
+                </geometry>
+            </collision>
+            <visual>
+                <origin xyz="0 0 0" rpy="0 0 0"/>
+                <geometry>
+                    <mesh filename="package://rrbot_description/meshes/hokuyo.dae"/>
+                </geometry>
+            </visual>
+            <inertial>
+                <mass value="1e-5" />
+                <origin xyz="0 0 0" rpy="0 0 0"/>
+                <inertia ixx="1e-6" ixy="0" ixz="0" iyy="1e-6" iyz="0" izz="1e-6" />
+            </inertial>
+        </link>
+        <joint name="laser_joint_left" type="fixed">
+            <!-- <origin xyz="0.0 0.25 0.29" rpy="-0.5 0 0"/> -->
+            <origin xyz="0.0 0.25 -0.20" rpy="0 0.01 ${3.14/2}"/>
+            <parent link="chasis"/>
+            <child link="hokuyo_link_left"/>
+        </joint>
+    </xacro:macro>
+    <!-- Hokuyo Laser - RIGHT -->
+    <xacro:macro name="laser_right">
+        <gazebo reference="hokuyo_link_right">
+            <sensor type="ray" name="head_hokuyo_sensor_right">
+            <pose>0 0 0 0 0 0</pose>
+            <visualize>true</visualize>
+            <update_rate>20</update_rate>
+            <ray>
+                <scan>
+                    <horizontal>
+                        <samples>50</samples>
                         <resolution>1</resolution>
                         <!-- <min_angle>-1.570796</min_angle> -->
@@ -154,40 +218,39 @@
             </ray>
             <plugin name="gazebo_ros_head_hokuyo_controller" filename="libgazebo_ros_laser.so">
-                <topicName>/scan_left</topicName>
-                <frameName>hokuyo_link_left</frameName>
+                <topicName>/scan_right</topicName>
+                <frameName>hokuyo_link_right</frameName>
             </plugin>
             </sensor>
         </gazebo>
         <!--  -->
-        <link name="hokuyo_link_left">
-            <collision>
-                <origin xyz="0 0 0" rpy="0 0 0"/>
-                <geometry>
-                    <box size="0.1 0.1 0.1"/>
-                </geometry>
-            </collision>
-            <visual>
-                <origin xyz="0 0 0" rpy="0 0 0"/>
-                <geometry>
-                    <mesh filename="package://rrbot_description/meshes/hokuyo.dae"/>
-                </geometry>
-            </visual>
-            <inertial>
-                <mass value="1e-5" />
-                <origin xyz="0 0 0" rpy="0 0 0"/>
-                <inertia ixx="1e-6" ixy="0" ixz="0" iyy="1e-6" iyz="0" izz="1e-6" />
-            </inertial>
-        </link>
-        <joint name="laser_joint_left" type="fixed">
-            <!-- <origin xyz="0.0 0.25 0.29" rpy="-0.5 0 0"/> -->
-            <origin xyz="0.0 0.25 -0.20" rpy="0 0.01 ${3.14/2}"/>
-            <parent link="chasis"/>
-            <child link="hokuyo_link_left"/>
-        </joint>
-    </xacro:macro>
-    <!-- Hokuyo Laser - RIGHT -->
-    <xacro:macro name="laser_right">
-        <gazebo reference="hokuyo_link_right">
-            <sensor type="ray" name="head_hokuyo_sensor_right">
+        <link name="hokuyo_link_right">
+            <collision>
+                <origin xyz="0 0 0" rpy="0 0 0"/>
+                <geometry>
+                    <box size="0.1 0.1 0.1"/>
+                </geometry>
+            </collision>
+            <visual>
+                <origin xyz="0 0 0" rpy="0 0 0"/>
+                <geometry>
+                    <mesh filename="package://rrbot_description/meshes/hokuyo.dae"/>
+                </geometry>
+            </visual>
+            <inertial>
+                <mass value="1e-5" />
+                <origin xyz="0 0 0" rpy="0 0 0"/>
+                <inertia ixx="1e-6" ixy="0" ixz="0" iyy="1e-6" iyz="0" izz="1e-6" />
+            </inertial>
+        </link>
+        <joint name="laser_joint_right" type="fixed">
+            <origin xyz="0.0 -0.25 -0.20" rpy="0 0.01 -${3.14/2}"/>
+            <parent link="chasis"/>
+            <child link="hokuyo_link_right"/>
+        </joint>
+    </xacro:macro>
+    <!-- Hokuyo Laser - REAR -->
+    <xacro:macro name="laser_rear">
+        <gazebo reference="hokuyo_link_rear">
+            <sensor type="ray" name="head_hokuyo_sensor_rear">
             <pose>0 0 0 0 0 0</pose>
             <visualize>true</visualize>
@@ -216,65 +279,4 @@
             </ray>
             <plugin name="gazebo_ros_head_hokuyo_controller" filename="libgazebo_ros_laser.so">
-                <topicName>/scan_right</topicName>
-                <frameName>hokuyo_link_right</frameName>
-            </plugin>
-            </sensor>
-        </gazebo>
-        <!--  -->
-        <link name="hokuyo_link_right">
-            <collision>
-                <origin xyz="0 0 0" rpy="0 0 0"/>
-                <geometry>
-                    <box size="0.1 0.1 0.1"/>
-                </geometry>
-            </collision>
-            <visual>
-                <origin xyz="0 0 0" rpy="0 0 0"/>
-                <geometry>
-                    <mesh filename="package://rrbot_description/meshes/hokuyo.dae"/>
-                </geometry>
-            </visual>
-            <inertial>
-                <mass value="1e-5" />
-                <origin xyz="0 0 0" rpy="0 0 0"/>
-                <inertia ixx="1e-6" ixy="0" ixz="0" iyy="1e-6" iyz="0" izz="1e-6" />
-            </inertial>
-        </link>
-        <joint name="laser_joint_right" type="fixed">
-            <origin xyz="0.0 -0.25 -0.20" rpy="0 0.01 -${3.14/2}"/>
-            <parent link="chasis"/>
-            <child link="hokuyo_link_right"/>
-        </joint>
-    </xacro:macro>
-    <!-- Hokuyo Laser - REAR -->
-    <xacro:macro name="laser_rear">
-        <gazebo reference="hokuyo_link_rear">
-            <sensor type="ray" name="head_hokuyo_sensor_rear">
-            <pose>0 0 0 0 0 0</pose>
-            <visualize>true</visualize>
-            <update_rate>20</update_rate>
-            <ray>
-                <scan>
-                    <horizontal>
-                        <samples>720</samples>
-                        <resolution>1</resolution>
-                        <!-- <min_angle>-1.570796</min_angle> -->
-                        <!-- <max_angle>1.570796</max_angle> -->
-                        <min_angle>-1.5</min_angle>
-                        <max_angle>1.5</max_angle>
-                    </horizontal>
-                </scan>
-                <range>
-                    <min>0.10</min>
-                    <max>10.0</max>
-                    <resolution>0.05</resolution>
-                </range>
-                <noise>
-                    <type>gaussian</type>
-                    <mean>0.0</mean>
-                    <stddev>0.01</stddev>
-                </noise>
-            </ray>
-            <plugin name="gazebo_ros_head_hokuyo_controller" filename="libgazebo_ros_laser.so">
                 <topicName>/scan_rear</topicName>
                 <frameName>hokuyo_link_rear</frameName>
